Commit message: Launch file autonomy_demo.launch.py starts the APRIL tag, LiDAR, and navigator nodes, along with joint state and robot state publishers. Images from the camera and points from the LiDAR can be displayed simultaneously via rviz2, in a valid frame tree.
https://github.com/billmania/roboquest_addons/issues/14

File: urdf/rq_tracked.urdf (robot description, URDF)
Before this commit: robot rq_tracked, 2 links, 1 joints
Links:
- added link laser, mass 0.1; collision box size=0.05 0.05 0.1; visual box size=0.05 0.05 0.1
Joints:
- added joint laser_base_joint: type fixed, parent base_link, child laser, origin xyz=0.25 0 0 rpy=0 0 0, limit effort=1 velocity=20
- joint camera_base_joint: origin xyz=0.25 0 0.15 rpy=0 0 0 -> xyz=0.15 0 0.15 rpy=0 0 0
